Commit message: [name edit]

File: roomiearm_description/gazebo/roomie_4dof.gazebo.xacro (robot description, xacro)
@@ -1,9 +1,9 @@
 <?xml version="1.0"?>
 <robot xmlns:xacro="http://ros.org/wiki/xacro">
-  <xacro:macro name="roomie_4dof_gazebo" params="prefix">
+  <xacro:macro name="roomiearm_4dof_gazebo" params="prefix">
     <!-- ros2_control Gazebo 플러그인 -->
     <gazebo>
       <plugin filename="libgz_ros2_control-system.so" name="gz_ros2_control::GazeboSimROS2ControlPlugin">
-        <parameters>$(find arm_gazebo)/config/roomie_controllers.yaml</parameters>
+        <parameters>$(find roomiearm_gazebo)/config/roomie_controllers.yaml</parameters>
         <robot_param>robot_description</robot_param>
         <robot_param_node>robot_state_publisher</robot_param_node>
@@ -17,5 +17,5 @@
         <update_rate>30.0</update_rate>
         <topic>camera/image_raw</topic>
-        <camera name="arm_camera">
+        <camera name="roomiearm_camera">
           <camera_info_topic>camera/camera_info</camera_info_topic>
           <horizontal_fov>1.0466</horizontal_fov>

File: roomiearm_description/ros2_control/roomie_4dof.ros2_control.xacro (robot description, xacro)
@@ -1,5 +1,5 @@
 <?xml version="1.0"?>
 <robot xmlns:xacro="http://www.ros.org/wiki/xacro">
-  <xacro:macro name="roomie_4dof_ros2_control" params="name prefix use_gazebo:=^|false">
+  <xacro:macro name="roomiearm_4dof_ros2_control" params="name prefix use_gazebo:=false">
     <ros2_control name="${name}" type="system">
       <hardware>
@@ -9,5 +9,5 @@
         <xacro:unless value="${use_gazebo}">
           <!-- 실제 하드웨어용 플러그인 (나중에 구현) -->
-          <plugin>roomie_ac/RoomieHardwareInterface</plugin>
+          <plugin>roomiearm_ac/RoomieHardwareInterface</plugin>
           <param name="serial_port">/dev/ttyUSB0</param>
           <param name="baudrate">115200</param>

File: roomiearm_description/urdf/roomie_4dof.xacro (robot description, xacro)
@@ -1,8 +1,8 @@
 <?xml version="1.0"?>
-<robot name="roomie_4dof" xmlns:xacro="http://www.ros.org/wiki/xacro">
+<robot name="roomiearm_4dof" xmlns:xacro="http://www.ros.org/wiki/xacro">
   <!-- Arguments -->
   <xacro:arg name="use_gazebo" default="false"/>
   <!-- Properties -->
-  <xacro:property name="mesh_prefix" value="package://arm_description/meshes"/>
+  <xacro:property name="mesh_prefix" value="package://roomiearm_description/meshes"/>
   <xacro:property name="limit_lower" value="-1.54"/>
   <xacro:property name="limit_upper" value="1.54"/>
@@ -196,11 +196,11 @@
   <!-- ===================================================== -->
   <!-- ros2_control 매크로 include -->
-  <xacro:include filename="$(find arm_description)/ros2_control/roomie_4dof.ros2_control.xacro"/>
-  <xacro:include filename="$(find arm_description)/gazebo/roomie_4dof.gazebo.xacro"/>
+  <xacro:include filename="$(find roomiearm_description)/ros2_control/roomie_4dof.ros2_control.xacro"/>
+  <xacro:include filename="$(find roomiearm_description)/gazebo/roomie_4dof.gazebo.xacro"/>
   <!-- ros2_control 매크로 호출 -->
-  <xacro:roomie_4dof_ros2_control name="RoomieSystem" prefix="" use_gazebo="$(arg use_gazebo)"/>
+  <xacro:roomiearm_4dof_ros2_control name="RoomieSystem" prefix="" use_gazebo="$(arg use_gazebo)"/>
   <xacro:if value="$(arg use_gazebo)">
     <!-- Gazebo 사용시만 포함 -->
-    <xacro:roomie_4dof_gazebo prefix=""/>
+    <xacro:roomiearm_4dof_gazebo prefix=""/>
   </xacro:if>
 </robot>
