Commit message: [camera.urdf.xacro수정]

File: roomiearm_description/urdf/mech/arm.urdf.xacro (robot description, xacro)
@@ -96,4 +96,5 @@
         <geometry><mesh filename="${mesh_prefix}/camera.stl"/></geometry>
         <material name="black"/>
+        <origin xyz="0 0 0" rpy="0 ${pi/2} 0"/>
       </visual>
       <collision>
@@ -151,11 +152,11 @@
     <parent link='link_4'/>
     <child link='camera_mount'/>
-    <origin xyz="-0.0035 0 0.054" rpy="0 0 0"/>
+    <origin xyz="-0.0035 0 0.054" rpy="0 -${pi/2} 0"/>
   </joint>
   <!-- Camera Optical Joint -->
   <joint name="camera_optical_joint" type="fixed">
-    <parent link="camera_link_mount"/>
+    <parent link="camera_mount"/>
     <child link="camera_link"/>
-    <origin xyz="0 0 0.01" rpy="0 0 ${-pi/2}"/>
+    <origin xyz="0.01 0 0" rpy="-${pi/2} 0 -${pi/2}"/>
   </joint>
 </robot>

File: roomiearm_description/urdf/mech/base.urdf.xacro (robot description, xacro)
@@ -1,5 +1,5 @@
 <?xml version="1.0" ?>
 <robot xmlns:xacro="http://wiki.ros.org/xacro">
-    <xacro:macro name="base" params="base_link prefix">
+    <xacro:macro name="base" params="base_link">
         <link name="base_link">
             <inertial>
@@ -12,5 +12,7 @@
             </inertial>
             <visual>
-                <geometry><mesh filename="${mesh_prefix}/base_link.stl"/></geometry>
+                <geometry>
+                    <mesh filename="file://$(find roomiearm_description)/meshes/base_link.stl"/>
+                </geometry>
                 <material name="grey"/>
             </visual>
@@ -22,5 +24,5 @@
             </collision>
         </link>
-        <gazebo reference="${prefix}${base_link}">
+        <gazebo reference="${base_link}">
             <visual>
                 <material>

File: roomiearm_description/urdf/robots/roomiearm.urdf.xacro (robot description, xacro)
@@ -3,12 +3,12 @@
     <xacro:arg name="robot_name" default="roomiearm"/>
     <xacro:arg name="add_world" default="true"/>
-    <xacro:arg name="prefix" default=""/>
-    <xacro:arg name="use_camera" default="false"/>
+    <xacro:arg name="base_link" default="base_link"/>
+    <xacro:arg name="base_type" default="g_shape"/>
     <xacro:arg name="use_gazebo" default="false"/>
     <xacro:if value="$(arg add_world)">
       <link name="world"/>
-      <joint name="$(arg prefix)virtual_joint" type="fixed">
+      <joint name="virtual_joint" type="fixed">
           <parent link="world"/>
-          <child link="$(arg prefix)$(arg base_link)"/>
+          <child link="$(arg base_link)"/>
           <origin xyz="0 0 0" rpy="0 0 0"/>
       </joint>
@@ -16,37 +16,17 @@
     <xacro:property name="current_base" value="$(arg base_type)"/>
     <xacro:if value="${current_base == 'g_shape'}">
-        <xacro:include filename="$(find roomiearm_description)/urdf/mech/g_shape_base_v2_0.urdf.xacro"/>
-        <xacro:g_shape_base
-            base_link="$(arg base_link)"
-            prefix="$(arg prefix)"/>
+        <xacro:include filename="$(find roomiearm_description)/urdf/mech/base.urdf.xacro"/>
+        <xacro:base base_link="$(arg base_link)"/>
     </xacro:if>
-    <xacro:include filename="$(find roomiearm_description)/urdf/mech/roomiearm_280_arm.urdf.xacro"/>
-    <xacro:roomiearm_280_arm
-      base_link="$(arg base_link)"
-      flange_link="$(arg flange_link)"
-      prefix="$(arg prefix)">
-      <origin xyz="0 0 0" rpy="0 0 0"/>
-    </xacro:roomiearm_280_arm>
+    <xacro:include filename="$(find roomiearm_description)/urdf/mech/arm.urdf.xacro"/>
+    <xacro:roomiearm_arm
+      base_link="$(arg base_link)">
+    </xacro:roomiearm_arm>
     <xacro:include filename="$(find roomiearm_description)/urdf/control/gazebo_sim_ros2_control.urdf.xacro" />
     <xacro:load_gazebo_sim_ros2_control_plugin
-      robot_name="$(arg robot_name)"
       use_gazebo="$(arg use_gazebo)"/>
-    <xacro:include filename="$(find roomiearm_description)/urdf/control/roomiearm__control.urdf.xacro" />
+    <xacro:include filename="$(find roomiearm_description)/urdf/control/roomiearm_ros2_control.urdf.xacro" />
     <xacro:roomiearm_ros2_control
-      prefix="$(arg prefix)"
-      flange_link="$(arg flange_link)"
       use_gazebo="$(arg use_gazebo)"/>
     <xacro:include filename="$(find roomiearm_description)/urdf/sensors/camera.urdf.xacro"/>
-    <!-- ===================================================== -->
-    <!-- ================= ROS2_CONTROL ==================== -->
-    <!-- ===================================================== -->
-    <!-- ros2_control 매크로 include -->
-    <xacro:include filename="$(find roomiearm_description)/ros2_control/roomie_4dof.ros2_control.xacro"/>
-    <xacro:include filename="$(find roomiearm_description)/gazebo/roomie_4dof.gazebo.xacro"/>
-    <!-- ros2_control 매크로 호출 -->
-    <xacro:roomiearm_4dof_ros2_control name="RoomieSystem" prefix="" use_gazebo="$(arg use_gazebo)"/>
-    <xacro:if value="$(arg use_gazebo)">
-      <!-- Gazebo 사용시만 포함 -->
-      <xacro:roomiearm_4dof_gazebo prefix=""/>
-    </xacro:if>
 </robot>
