Commit message: [roomie_core 리팩토링]

File: roomiearm_description/urdf/control/roomiearm_ros2_control.urdf.xacro (robot description, xacro)
@@ -1,42 +1,39 @@
 <?xml version="1.0"?>
 <robot xmlns:xacro="http://www.ros.org/wiki/xacro">
-  <xacro:macro name="roomiearm_ros2_control" params="use_gazebo">
-    <ros2_control name="RobotSystem" type="system">
+  <xacro:macro name="roomiearm_ros2_control" params="name:=RoomieArm use_gazebo:=false">
+    <ros2_control name="${name}" type="system">
       <hardware>
         <xacro:if value="${use_gazebo}">
-           <plugin>gz_ros2_control/GazeboSimSystem</plugin>
+          <plugin>gz_ros2_control/GazeboSimSystem</plugin>
         </xacro:if>
+        <xacro:unless value="${use_gazebo}">
+          <plugin>roomiearm_hardware/RoomieArmHardwareInterface</plugin>
+          <param name="serial_port_name">/dev/ttyACM0</param>
+          <param name="serial_baud_rate">115200</param>
+        </xacro:unless>
       </hardware>
-      <!-- Joint 1 -->
       <joint name="joint_1">
-        <command_interface name="position">
-          <param name="min">-1.5708</param>
-          <param name="max">1.5708</param>
-        </command_interface>
+        <command_interface name="position"/>
+        <command_interface name="velocity"/>
         <state_interface name="position"/>
+        <state_interface name="velocity"/>
       </joint>
-      <!-- Joint 2 -->
       <joint name="joint_2">
-        <command_interface name="position">
-          <param name="min">-1.5708</param>
-          <param name="max">1.5708</param>
-        </command_interface>
+        <command_interface name="position"/>
+        <command_interface name="velocity"/>
         <state_interface name="position"/>
+        <state_interface name="velocity"/>
       </joint>
-      <!-- Joint 3 -->
       <joint name="joint_3">
-        <command_interface name="position">
-          <param name="min">-1.5708</param>
-          <param name="max">1.5708</param>
-        </command_interface>
+        <command_interface name="position"/>
+        <command_interface name="velocity"/>
         <state_interface name="position"/>
+        <state_interface name="velocity"/>
       </joint>
-      <!-- Joint 4 -->
       <joint name="joint_4">
-        <command_interface name="position">
-          <param name="min">-1.5708</param>
-          <param name="max">1.5708</param>
-        </command_interface>
+        <command_interface name="position"/>
+        <command_interface name="velocity"/>
         <state_interface name="position"/>
+        <state_interface name="velocity"/>
       </joint>
     </ros2_control>

File: roomiearm_description/urdf/sensors/camera.urdf.xacro (robot description, xacro)
@@ -13,6 +13,6 @@
             <horizontal_fov>1.0466</horizontal_fov>
             <image>
-              <width>800</width>
-              <height>600</height>
+              <width>640</width>
+              <height>480</height>
               <format>R8G8B8</format>
             </image>
@@ -21,12 +21,4 @@
               <far>300</far>
             </clip>
-            <distortion>
-              <k1>-0.414921465</k1>
-              <k2>0.277976117</k2>
-              <p1>0.000362302582</p1>
-              <p2>-0.000173492775</p2>
-              <k3>-0.194112104</k3>
-              <center>0.5 0.5</center>
-            </distortion>
             <noise>
             <type>gaussian</type>
